Commit message: teleoperate추가

File: urdf/two_arm_URDF_fixed.urdf (robot description, URDF)
Before this commit: robot two_arm_URDF, 13 links, 12 joints
Links:
- link base: geometry collision mesh filename=package://final_project_two_arm/meshes/base.stl scale=1.0 1.0 1.0; visual mesh filename=package://final_project_two_arm/meshes/base.stl scale=1.0 1.0 1.0
- link end_point_L: geometry collision mesh filename=package://final_project_two_arm/meshes/end_point_L.stl scale=1.0 1.0 1.0; visual mesh filename=package://final_project_two_arm/meshes/end_point_L.stl scale=1.0 1.0 1.0
- link end_point_R: geometry collision mesh filename=package://final_project_two_arm/meshes/end_point_R.stl scale=1.0 1.0 1.0; visual mesh filename=package://final_project_two_arm/meshes/end_point_R.stl scale=1.0 1.0 1.0
- link link_1_L: geometry collision mesh filename=package://final_project_two_arm/meshes/link_1_L.stl scale=1.0 1.0 1.0; visual mesh filename=package://final_project_two_arm/meshes/link_1_L.stl scale=1.0 1.0 1.0
- link link_1_R: geometry collision mesh filename=package://final_project_two_arm/meshes/link_1_R.stl scale=1.0 1.0 1.0; visual mesh filename=package://final_project_two_arm/meshes/link_1_R.stl scale=1.0 1.0 1.0
- link link_2_L: geometry collision mesh filename=package://final_project_two_arm/meshes/link_2_L.stl scale=1.0 1.0 1.0; visual mesh filename=package://final_project_two_arm/meshes/link_2_L.stl scale=1.0 1.0 1.0
- link link_2_R: geometry collision mesh filename=package://final_project_two_arm/meshes/link_2_R.stl scale=1.0 1.0 1.0; visual mesh filename=package://final_project_two_arm/meshes/link_2_R.stl scale=1.0 1.0 1.0
- link link_3_L: geometry collision mesh filename=package://final_project_two_arm/meshes/link_3_L.stl scale=1.0 1.0 1.0; visual mesh filename=package://final_project_two_arm/meshes/link_3_L.stl scale=1.0 1.0 1.0
- link link_3_R: geometry collision mesh filename=package://final_project_two_arm/meshes/link_3_R.stl scale=1.0 1.0 1.0; visual mesh filename=package://final_project_two_arm/meshes/link_3_R.stl scale=1.0 1.0 1.0
- link link_4_L: geometry collision mesh filename=package://final_project_two_arm/meshes/link_4_L.stl scale=1.0 1.0 1.0; visual mesh filename=package://final_project_two_arm/meshes/link_4_L.stl scale=1.0 1.0 1.0
- link link_4_R: geometry collision mesh filename=package://final_project_two_arm/meshes/link_4_R.stl scale=1.0 1.0 1.0; visual mesh filename=package://final_project_two_arm/meshes/link_4_R.stl scale=1.0 1.0 1.0
- link link_5_L: geometry collision mesh filename=package://final_project_two_arm/meshes/link_5_L.stl scale=1.0 1.0 1.0; visual mesh filename=package://final_project_two_arm/meshes/link_5_L.stl scale=1.0 1.0 1.0
- link link_5_R: geometry collision mesh filename=package://final_project_two_arm/meshes/link_5_R.stl scale=1.0 1.0 1.0; visual mesh filename=package://final_project_two_arm/meshes/link_5_R.stl scale=1.0 1.0 1.0
Joints:
- joint rot_L1: limit lower=-3.1416 upper=3.1416 effort=10.0 velocity=0.35 -> lower=-3.1416 upper=3.1416 effort=10.0 velocity=0.34
- joint rot_L2: limit lower=-2.0944 upper=0.3491 effort=10.0 velocity=0.35 -> lower=-2.0944 upper=0.3491 effort=10.0 velocity=0.34
- joint rot_L3: limit lower=-3.1416 upper=3.1416 effort=10.0 velocity=1.0 -> lower=-3.1416 upper=3.1416 effort=10.0 velocity=1.02
- joint rot_L4: limit lower=-2.0944 upper=0.1745 effort=10.0 velocity=1.0 -> lower=-2.0944 upper=0.1745 effort=10.0 velocity=1.02
- joint rot_L5: limit lower=-3.1416 upper=3.1416 effort=10.0 velocity=3.0 -> lower=-3.1416 upper=3.1416 effort=10.0 velocity=5.11
- joint rot_L6: limit lower=-1.7453 upper=1.7453 effort=10.0 velocity=3.0 -> lower=-1.7453 upper=1.7453 effort=10.0 velocity=5.11
- joint rot_R1: limit lower=-3.1416 upper=3.1416 effort=10.0 velocity=0.35 -> lower=-3.1416 upper=3.1416 effort=10.0 velocity=0.34
- joint rot_R2: limit lower=-2.0944 upper=0.3491 effort=10.0 velocity=0.35 -> lower=-2.0944 upper=0.3491 effort=10.0 velocity=0.34
- joint rot_R3: limit lower=-3.1416 upper=3.1416 effort=10.0 velocity=1.0 -> lower=-3.1416 upper=3.1416 effort=10.0 velocity=1.02
- joint rot_R4: limit lower=-2.0944 upper=0.1745 effort=10.0 velocity=1.0 -> lower=-2.0944 upper=0.1745 effort=10.0 velocity=1.02
- joint rot_R5: limit lower=-3.1416 upper=3.1416 effort=10.0 velocity=3.0 -> lower=-3.1416 upper=3.1416 effort=10.0 velocity=5.11
- joint rot_R6: limit lower=-1.7453 upper=1.7453 effort=10.0 velocity=3.0 -> lower=-1.7453 upper=1.7453 effort=10.0 velocity=5.11

Commit message: Many fixed

File: urdf/two_arm_URDF_fixed.urdf (robot description, URDF)
Before this commit: robot two_arm_URDF, 13 links, 12 joints
Links:
- link base: geometry collision mesh filename=package://final_project_two_arm/meshes/base.stl scale=0.001 0.001 0.001; visual mesh filename=package://final_project_two_arm/meshes/base.stl scale=0.001 0.001 0.001
- link end_point_L: mass 1.8507809062204477 -> 2.238441847971124; geometry collision mesh filename=package://final_project_two_arm/meshes/end_point_L.stl scale=0.001 0.001 0.001; visual mesh filename=package://final_project_two_arm/meshes/end_point_L.stl scale=0.001 0.001 0.001
- link end_point_R: mass 1.850780774552443 -> 2.238439986935529; geometry collision mesh filename=package://final_project_two_arm/meshes/end_point_R.stl scale=0.001 0.001 0.001; visual mesh filename=package://final_project_two_arm/meshes/end_point_R.stl scale=0.001 0.001 0.001
- link link_1_L: geometry collision mesh filename=package://final_project_two_arm/meshes/link_1_L.stl scale=0.001 0.001 0.001; visual mesh filename=package://final_project_two_arm/meshes/link_1_L.stl scale=0.001 0.001 0.001
- link link_1_R: geometry collision mesh filename=package://final_project_two_arm/meshes/link_1_R.stl scale=0.001 0.001 0.001; visual mesh filename=package://final_project_two_arm/meshes/link_1_R.stl scale=0.001 0.001 0.001
- link link_2_L: geometry collision mesh filename=package://final_project_two_arm/meshes/link_2_L.stl scale=0.001 0.001 0.001; visual mesh filename=package://final_project_two_arm/meshes/link_2_L.stl scale=0.001 0.001 0.001
- link link_2_R: geometry collision mesh filename=package://final_project_two_arm/meshes/link_2_R.stl scale=0.001 0.001 0.001; visual mesh filename=package://final_project_two_arm/meshes/link_2_R.stl scale=0.001 0.001 0.001
- link link_3_L: geometry collision mesh filename=package://final_project_two_arm/meshes/link_3_L.stl scale=0.001 0.001 0.001; visual mesh filename=package://final_project_two_arm/meshes/link_3_L.stl scale=0.001 0.001 0.001
- link link_3_R: geometry collision mesh filename=package://final_project_two_arm/meshes/link_3_R.stl scale=0.001 0.001 0.001; visual mesh filename=package://final_project_two_arm/meshes/link_3_R.stl scale=0.001 0.001 0.001
- link link_4_L: geometry collision mesh filename=package://final_project_two_arm/meshes/link_4_L.stl scale=0.001 0.001 0.001; visual mesh filename=package://final_project_two_arm/meshes/link_4_L.stl scale=0.001 0.001 0.001
- link link_4_R: geometry collision mesh filename=package://final_project_two_arm/meshes/link_4_R.stl scale=0.001 0.001 0.001; visual mesh filename=package://final_project_two_arm/meshes/link_4_R.stl scale=0.001 0.001 0.001
- link link_5_L: geometry collision mesh filename=package://final_project_two_arm/meshes/link_5_L.stl scale=0.001 0.001 0.001; visual mesh filename=package://final_project_two_arm/meshes/link_5_L.stl scale=0.001 0.001 0.001
- link link_5_R: geometry collision mesh filename=package://final_project_two_arm/meshes/link_5_R.stl scale=0.001 0.001 0.001; visual mesh filename=package://final_project_two_arm/meshes/link_5_R.stl scale=0.001 0.001 0.001
Joints:
- joint rot_L1: axis 0.0 0.0 1.0 -> -4.1663675001976565e-32 3.8857805861880464e-16 1.0
- joint rot_L2: axis 0.0 0.0 1.0 -> -0.939693 9.299886998271218e-32 0.3420199999999999; origin xyz=0.039624999999999994 2.997602166487923e-17 0.07780000000000005 rpy=1.5707963267948966 -3.8857805861880464e-16 -1.5707963267948966 -> xyz=0.013552550000000005 -0.03723531999999997 0.07780000000000005 rpy=1.5707963267948966 -3.8857805861880464e-16 -1.5707963267948966
- joint rot_L3: axis 0.0 0.0 1.0 -> 0.939693 2.1078609906538316e-33 0.34202; origin xyz=-0.16125 0.0 0.039624999999999994 rpy=-3.141592653589793 1.5707963267948966 0 -> xyz=-0.09238606999999999 0.0 -0.13797288 rpy=-3.141592653589793 1.5707963267948966 0
- joint rot_L4: axis 0.0 0.0 1.0 -> 0.0 7.771561172376089e-16 1.0; origin xyz=0.0 0.03800000000000004 0.058750000000000004 rpy=1.5707963267948974 -0.0 -1.6605463961890884e-31 -> xyz=0.05520695 0.03800000000000004 0.020093680000000003 rpy=1.5707963267948974 -1.1102230246251565e-16 5.473822126268817e-48
- joint rot_L5: axis 0.0 0.0 1.0 -> 0.49999999999999994 0.0 -0.866025; origin xyz=0.0 0.18125000000000005 0.0379999999999999 rpy=-1.5707963267948974 -2.8037623946618293e-32 2.1789610962922083e-47 -> xyz=0.090625 -0.15696709999999997 0.038000000000000186 rpy=-1.5707963267948974 -4.733165431326071e-30 0.0
- joint rot_L6: axis 0.0 0.0 1.0 -> 0.0 7.771561172376101e-16 1.0; origin xyz=0.0 0.01900000000000006 0.04875 rpy=1.5707963267948974 -0.0 1.3481509610798863e-31 -> xyz=0.024375 0.01900000000000006 -0.04221874 rpy=1.5707963267948974 5.551115123125783e-17 4.733165431326072e-30
- joint rot_R1: axis 0.0 0.0 1.0 -> -4.1663675001976565e-32 -3.8857805861880464e-16 1.0
- joint rot_R2: axis 0.0 0.0 1.0 -> 0.939693 -3.1354432147666987e-32 0.34202; origin xyz=0.039624999999999994 3.053113317719181e-17 -0.07780000000000001 rpy=-1.5707963267948966 3.8857805861880464e-16 -1.5707963267948966 -> xyz=0.013552550000000005 -0.03723531999999997 -0.07780000000000002 rpy=-1.5707963267948966 3.8857805861880464e-16 -1.5707963267948968
- joint rot_R3: axis 0.0 0.0 -1.0 -> -0.939693 -2.1036110025269536e-32 -0.34202; origin xyz=-0.16125 0.0 -0.039624999999999994 rpy=-2.7143969068027984e-64 -1.5707963267948966 0 -> xyz=-0.09238607 0.0 0.13797288 rpy=1.2325951644078305e-32 -1.5707963267948966 0
- joint rot_R4: axis 0.0 0.0 -1.0 -> 0.0 7.771561172376087e-16 -1.0; origin xyz=0.0 -0.038000000000000006 0.058750000000000004 rpy=-1.5707963267948974 2.465190328815662e-32 9.935591755726858e-32 -> xyz=0.05520695 -0.038000000000000006 0.020093679999999996 rpy=-1.5707963267948974 -3.646298014371764e-63 4.930380657631325e-32
- joint rot_R5: axis 0.0 0.0 -1.0 -> -0.5 1.9438321565550953e-30 0.866025; origin xyz=0.0 -0.18125 0.03799999999999986 rpy=1.5707963267948974 -8.218831152865144e-32 -2.4651903288156685e-32 -> xyz=0.090625 0.15696709999999997 0.038000000000000124 rpy=1.5707963267948974 -0.0 0.0
- joint rot_R6: axis 0.0 0.0 -1.0 -> -3.1554436208840472e-30 7.771561172376069e-16 -1.0; origin xyz=0.0 -0.019000000000000003 0.04875 rpy=-1.5707963267948974 -0.0 -2.344225386936698e-31 -> xyz=0.024375 -0.019000000000000003 -0.04221874 rpy=-1.5707963267948974 5.551115123125783e-17 3.1554436208840472e-30
