Commit message: moveit2 success

File: urdf/two_arm_ver2.urdf (robot description, URDF)
Before this commit: robot arm_ver4_urdf, 15 links, 14 joints
Links:
- link base: mass 32.55922417276492 -> None
Joints:
- joint L_3: limit lower=-3.1416 upper=3.1416 effort=10.0 velocity=1.02 -> lower=-3.1416 upper=3.1416 effort=10.0 velocity=0.32
- joint L_4: limit lower=-2.0944 upper=0.1745 effort=10.0 velocity=1.02 -> lower=-2.0944 upper=0.1745 effort=10.0 velocity=0.32
- joint L_5: limit lower=-3.1416 upper=3.1416 effort=10.0 velocity=5.11 -> lower=-3.1416 upper=3.1416 effort=10.0 velocity=0.32
- joint L_6: limit lower=-1.7453 upper=1.7453 effort=10.0 velocity=5.11 -> lower=-1.7453 upper=1.7453 effort=10.0 velocity=0.32
- joint L_7: limit lower=-3.1416 upper=3.1416 effort=10.0 velocity=5.11 -> lower=-3.1416 upper=3.1416 effort=10.0 velocity=0.32
- joint R_3: limit lower=-3.1416 upper=3.1416 effort=10.0 velocity=1.02 -> lower=-3.1416 upper=3.1416 effort=10.0 velocity=0.32
- joint R_4: limit lower=-2.0944 upper=0.1745 effort=10.0 velocity=1.02 -> lower=-2.0944 upper=0.1745 effort=10.0 velocity=0.32
- joint R_5: limit lower=-3.1416 upper=3.1416 effort=10.0 velocity=5.11 -> lower=-3.1416 upper=3.1416 effort=10.0 velocity=0.32
- joint R_6: limit lower=-1.7453 upper=1.7453 effort=10.0 velocity=5.11 -> lower=-1.7453 upper=1.7453 effort=10.0 velocity=0.32
- joint R_7: limit lower=-3.1416 upper=3.1416 effort=10.0 velocity=5.11 -> lower=-3.1416 upper=3.1416 effort=10.0 velocity=0.32

Commit message: semi complete video

File: urdf/two_arm_ver2.urdf (robot description, URDF)
Before this commit: robot arm_ver4_urdf, 15 links, 14 joints
Joints:
- joint L_3: limit lower=-3.1416 upper=3.1416 effort=10.0 velocity=0.32 -> lower=-3.1416 upper=3.1416 effort=10.0 velocity=0.40
- joint R_3: limit lower=-3.1416 upper=3.1416 effort=10.0 velocity=0.32 -> lower=-3.1416 upper=3.1416 effort=10.0 velocity=0.40
